File: hardware/ABK-20.sch (KiCad schematic (older format))
At the start: 55 parts, among them J1 CONN_01X04, J2 CONN_01X04, J3 CONN_02X03, J4 Con_3-5V, J5 USB_OTG, J6 Sync_Jumper, SW1 SW_Push, SW2 SW_Push, SW3 SW_Push, SW4 SW_Push, U1 ATTINY85-20SU, U2 PAM8002, U3 7805

Commit message: Fix KiCad 5 to KiCad 9 symbol migration: upgrade cache symbols to kicad_sym and remap components
Parts:
- BT1, BT2: symbol Battery_Cell -> ABK-20-rescue:Battery_Cell
- C1, C2, C3, C4, C5, C6: symbol C -> ABK-20-rescue:C
- C7: symbol CP -> ABK-20-rescue:CP
- D-OUT1, D-POW1: symbol LED -> ABK-20-rescue:LED
- J1, J2: symbol CONN_01X04 -> ABK-20-rescue:CONN_01X04
- J3: symbol CONN_02X03 -> ABK-20-rescue:CONN_02X03
- J4: symbol CONN_01X02 -> ABK-20-rescue:CONN_01X02
- J5: symbol USB_OTG -> ABK-20-rescue:USB_OTG
- J6: symbol CONN_01X02_MALE -> ABK-20-rescue:CONN_01X02_MALE
- Jack1, Jack2: symbol JACK_TRS_6PINS -> ABK-20-rescue:JACK_TRS_6PINS
- NEO1, NEO2, NEO3, NEO4, NEO5, NEO6, NEO7, NEO8: symbol SK6812 -> ABK-20-rescue:SK6812
- POT1-MAIN1, POT2-CV1, POT3-Vol1: symbol POT -> ABK-20-rescue:POT
- R1, R10, R11, R12, R13, R14, R15, R2, R3, R4, R5, R6, R7, R8, R9, R99: symbol R -> ABK-20-rescue:R
- SW1, SW2, SW3, SW4: symbol SW_Push -> ABK-20-rescue:SW_Push
- Speaker1: symbol Speaker -> ABK-20-rescue:Speaker
- U1: symbol ATTINY85-20SU -> ABK-20-rescue:ATTINY85-20SU
- U2: symbol PAM8002 -> ABK-20-rescue:PAM8002
- U3: footprint TO_SOT_Packages_SMD:TO-252-3_TabPin2 -> Package_TO_SOT_SMD:TO-252-3_TabPin2; symbol 7805 -> ABK-20-rescue:7805
- board1: symbol CONN_01X01 -> ABK-20-rescue:CONN_01X01

Commit message: Update sym-lib-table with ABK-20-rescue kicad_sym mapping
Parts:
- U3: footprint Package_TO_SOT_SMD:TO-252-3_TabPin2 -> TO_SOT_Packages_SMD:TO-252-3_TabPin2
Changed lines of the file:
@@
 LIBS:contrib
 LIBS:valves
-LIBS:MixtapeNEO-3000-cache
+LIBS:ABK-20-cache
 EELAYER 25 0
 EELAYER END
@@
 F 0 "U3" H 1550 1004 50  0000 C CNN
 F 1 "7805" H 1400 1400 50  0000 C CNN
-F 2 "Package_TO_SOT_SMD:TO-252-3_TabPin2" H 1400 1200 50  0001 C CNN
+F 2 "TO_SOT_Packages_SMD:TO-252-3_TabPin2" H 1400 1200 50  0001 C CNN
 F 3 "" H 1400 1200 50  0001 C CNN
 	1    1400 1200
