File: hardware/ABK-20.sch (KiCad schematic (older format))
At the start: 55 parts, among them J1 CONN_01X04, J2 CONN_01X04, J3 CONN_02X03, J4 Con_3-5V, J5 USB_OTG, J6 Sync_Jumper, SW1 SW_Push, SW2 SW_Push, SW3 SW_Push, SW4 SW_Push, U1 ATTINY85-20SU, U2 PAM8002, U3 7805

Commit message: Restore clean unprefixed KiCad 4 schematic ready for Remap Symbols dialog
Parts:
- BT1, BT2: symbol ABK-20-rescue:Battery_Cell -> Battery_Cell
- C1, C2, C3, C4, C5, C6: symbol ABK-20-rescue:C -> C
- C7: symbol ABK-20-rescue:CP -> CP
- D-OUT1, D-POW1: symbol ABK-20-rescue:LED -> LED
- J1, J2: symbol ABK-20-rescue:CONN_01X04 -> CONN_01X04
- J3: symbol ABK-20-rescue:CONN_02X03 -> CONN_02X03
- J4: symbol ABK-20-rescue:CONN_01X02 -> CONN_01X02
- J5: symbol ABK-20-rescue:USB_OTG -> USB_OTG
- J6: symbol ABK-20-rescue:CONN_01X02_MALE -> CONN_01X02_MALE
- Jack1, Jack2: symbol ABK-20-rescue:JACK_TRS_6PINS -> JACK_TRS_6PINS
- NEO1, NEO2, NEO3, NEO4, NEO5, NEO6, NEO7, NEO8: symbol ABK-20-rescue:SK6812 -> SK6812
- POT1-MAIN1, POT2-CV1, POT3-Vol1: symbol ABK-20-rescue:POT -> POT
- R1, R10, R11, R12, R13, R14, R15, R2, R3, R4, R5, R6, R7, R8, R9, R99: symbol ABK-20-rescue:R -> R
- SW1, SW2, SW3, SW4: symbol ABK-20-rescue:SW_Push -> SW_Push
- Speaker1: symbol ABK-20-rescue:Speaker -> Speaker
- U1: symbol ABK-20-rescue:ATTINY85-20SU -> ATTINY85-20SU
- U2: symbol ABK-20-rescue:PAM8002 -> PAM8002
- U3: symbol ABK-20-rescue:7805 -> 7805
- board1: symbol ABK-20-rescue:CONN_01X01 -> CONN_01X01
