File: hardware/LED_Matrix.kicad_sch (KiCad schematic)
At the start: 21 parts

Commit message: feat(hardware): complete 75x80 mm PCB routing, interactive BOM, 3D models and gerbers
Parts:
- R9: footprint 8Bitmixtape_reworked:R_1206_HandSoldering -> 007_dusjagr:R_1206_noGND_sm
Changed lines of the file:
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@@
 			)
 		)
-		(property "Footprint" "8Bitmixtape_reworked:R_1206_HandSoldering"
+		(property "Footprint" "007_dusjagr:R_1206_noGND_sm"
 			(at 97.79 57.222 90)
 			(effects
